Commit message: remove the old imu, update readme

File: robots/descriptions/go2_description/xacro/gazebo.xacro (robot description, xacro)
@@ -19,5 +19,5 @@
       </plugin>
     </gazebo>
-    <gazebo reference="imu_link">
+    <!-- <gazebo reference="imu_link">
         <sensor name="imu_sensor" type="imu">
             <always_on>true</always_on>
@@ -73,5 +73,5 @@
             </plugin>
         </sensor>
-    </gazebo>
+    </gazebo> -->
     <!-- <gazebo reference="base_link">
         <turnGravityOff>false</turnGravityOff>

File: robots/descriptions/go2_description/xacro/robot_VLP.xacro (robot description, xacro)
@@ -56,5 +56,5 @@
         </inertial>
     </link>
-    <joint name="imu_joint" type="fixed">
+    <!-- <joint name="imu_joint" type="fixed">
         <parent link="trunk"/>
         <child link="imu_link"/>
@@ -79,5 +79,5 @@
             </geometry>
         </collision>
-    </link>
+    </link> -->
     <!--
     <joint name="load_joint" type="fixed">
