Commit message: update go2w frame names

File: robots/descriptions/go2w_description/urdf/go2w_description.urdf.xacro (robot description, xacro)
@@ -223,5 +223,5 @@
   </xacro:macro>
   <!-- Base-->
-  <link name="base"/>
+  <link name="base_link"/>
   <!-- Body -->
   <link name="body">
@@ -245,5 +245,5 @@
   </link>
   <joint name="body_joint" type="fixed">
-    <parent link="base" />
+    <parent link="base_link" />
     <child link="body" />
   </joint>
@@ -293,5 +293,5 @@
   <xacro:leg prefix="RR" front="False" left="False"/>
   <!-- IMU -->
-  <link name="imu">
+  <!-- <link name="imu">
     <inertial>
       <origin xyz="0 0 0" rpy="0 0 0" />
@@ -361,7 +361,7 @@
       </plugin>
     </sensor>
-  </gazebo>
+  </gazebo> -->
   <!-- Lidar -->
-  <link name="lidar">
+  <!-- <link name="lidar">
     <inertial>
       <origin xyz="0 0 0" rpy="0 0 0" />
@@ -415,5 +415,5 @@
       </plugin>
     </sensor>
-  </gazebo>
+  </gazebo> -->
   <!-- =============== mid360 ============ -->
   <!-- <origin xyz="0.3 0.0 0.10" rpy="0 0.5235987756 0"/> -->
@@ -553,6 +553,6 @@
       <origin xyz="-0.1 0 0.06" rpy="0 0 0"/>
   </xacro:gps_sensor>
-  <xacro:mid360 name="livox" parent="body">
-      <origin xyz="0 0 0.10" rpy="0 0 0"/>
+  <xacro:mid360 name="livox_frame" parent="body">
+      <origin xyz="0.25 0 0.13" rpy="0 0.4 0"/>
   </xacro:mid360>
 </robot>
